Commit message: compare v3 vs baseline input sensitivity , command curriculum condition modified

File: humanoidverse/data/robots/g1/g1_29dof_anneal_23dof.urdf (robot description, URDF)
Before this commit: robot g1_29dof, 39 links, 38 joints
Joints:
- joint left_wrist_roll_joint: origin xyz=0.100 0.00188791 -0.010 rpy=0 0 0 -> xyz=0.100 0.00188791 -0.010 rpy=0.15 0 0
- joint right_wrist_roll_joint: origin xyz=0.100 -0.00188791 -0.010 rpy=0 0 0 -> xyz=0.100 -0.00188791 -0.010 rpy=-0.15 0 0
